Commit message: delete odom file

File: src/cartographer_ros/cartographer_ros/urdf/my_robot.urdf (robot description, URDF)
Before this commit: robot jd_robot, 5 links, 4 joints
Joints:
- joint gps_link_joint: origin xyz=-0.878521 -0.319632 0.0661 rpy=0 0 0 -> xyz=-0.878521 -0.319632 0.2035 rpy=0 0 0
